File: X13-Backplane.sch (EAGLE design)
At the start: 45 parts, among them J2 284512-4, J3 284512-8, J4 284512-8, J5 284512-4, Y1 ECS-80-S-4X

Commit message: Updated Solenoid Board
Parts:
- removed U$1, U$5, U$6: LV8548M, HBridge:LV8548M
- added U1: ULN2003V12, ULN2003V12:ULN2003V12
Connections:
- removed net GPIO0: U$1.IN4, U$3.PB7
- removed net SOL1_2: J1.1, U$1.OUT2
- removed net SOL2_2: J6.1, U$1.OUT4
- removed net SOL3_2: J7.1, U$5.OUT2
- removed net SOL4_2: J8.1, U$5.OUT4
- removed net SOL5_2: J9.1, U$6.OUT2
- removed net SOL6_2: J10.1, U$6.OUT4
- new net ALERT: U$3.PB7
- new net CLK: U$3.PA9
- new net DATA: U$3.PA10
- net 12V: now also J1.1, J10.1, J6.1, J7.1, J8.1, J9.1, U1.COM; no longer U$1.VCC, U$5.VCC, U$6.VCC
- net GND: now also U1.GND; no longer U$1.GND, U$5.GND, U$6.GND
- net GPIO1: now also U1.IN4; no longer U$1.IN3
- net GPIO10: now also U1.IN3; no longer U$5.IN3
- net GPIO11: now also U1.IN2; no longer U$5.IN4
- net GPIO12: now also U1.IN1; no longer U$6.IN1
- net GPIO13: no longer U$6.IN2
- net GPIO14: now also U$3.PA1; no longer U$3.PA9, U$6.IN3
- net GPIO15: now also U$3.PA0; no longer U$3.PA10, U$6.IN4
- net GPIO2: now also U1.IN5; no longer U$1.IN2
- net GPIO3: now also U1.IN6; no longer U$1.IN1
- net GPIO8: no longer U$5.IN1
- net GPIO9: no longer U$5.IN2
- net SOL1_1: now also U1.OUT1; no longer U$1.OUT1
- net SOL2_1: now also U1.OUT2; no longer U$1.OUT3
- net SOL3_1: now also U1.OUT3; no longer U$5.OUT1
- net SOL4_1: now also U1.OUT4; no longer U$5.OUT3
- net SOL5_1: now also U1.OUT5; no longer U$6.OUT1
- net SOL6_1: now also U1.OUT6; no longer U$6.OUT3
Other:
- note added: "NPN Array"
- note removed: "H-Bridges"
- moved on the sheet: C1, C10, C11, C18, C2, C3, C4, C5, C6, C7, C8, C9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

Commit message: added Thrusters/motor connectors + QuadESC Connectors
Parts:
- removed C18: 47uF, SparkFun-Capacitors:47UF-POLAR-PANASONIC_D-35V-20%
- removed J12: (no value), SparkFun-Connectors:CONN_02
- added MC1, MC2, MC3, MC4, T1, T2, T3, T4, T5, T6, T7, T8: 284512-3, ThrusterConnector:284512-3
- added U$1, U$4, U$5, U$6, U$7: ESC2BACKPLANE, ESC_to_Backplane_Connectors:ESC2BACKPLANE
- J11: value (none) -> 284512-8; device SparkFun-Connectors:CONN_02 -> 284512-8:284512-8
- U$2: value MURATA-DC-DC -> ESC2BACKPLANE; device MURATA_3pin_dcdc:MURATA-DC-DC -> ESC_to_Backplane_Connectors:ESC2BACKPLANE
Connections:
- new net ESC-ID_1: U$7G$1.P$8
- new net ESC-ID_2: U$5G$1.P$8
- new net ESC-ID_3: U$2G$1.P$8
- new net MC1_PHS1: MC1.P$1
- new net MC1_PHS2: MC1.P$2
- new net MC1_PHS3: MC1.P$3
- new net MC2_PHS1: MC2.P$1
- new net MC2_PHS2: MC2.P$2
- new net MC2_PHS3: MC2.P$3
- new net MC3_PHS1: MC3.P$1
- new net MC3_PHS2: MC3.P$2
- new net MC3_PHS3: MC3.P$3
- new net MC4_PHS1: MC4.P$1
- new net MC4_PHS2: MC4.P$2
- new net MC4_PHS3: MC4.P$3
- new net SWCLK_4: MUX.1Y3, U$3.PA14
- new net SWDIO_4: MUX.2Y3, U$3.PA13
- new net T1_PHS1: T1.P$1
- new net T1_PHS2: T1.P$2
- new net T1_PHS3: T1.P$3
- new net T2_PHS1: T2.P$1
- new net T2_PHS2: T2.P$2
- new net T2_PHS3: T2.P$3
- new net T3_PHS1: T3.P$1
- new net T3_PHS2: T3.P$2
- new net T3_PHS3: T3.P$3
- new net T4_PHS1: T4.P$1
- new net T4_PHS2: T4.P$2
- new net T4_PHS3: T4.P$3
- new net T5_PHS1: T5.P$1
- new net T5_PHS2: T5.P$2
- new net T5_PHS3: T5.P$3
- new net T6_PHS1: T6.P$1
- new net T6_PHS2: T6.P$2
- new net T6_PHS3: T6.P$3
- new net T7_PHS1: T7.P$1
- new net T7_PHS2: T7.P$2
- new net T7_PHS3: T7.P$3
- new net T8_PHS1: T8.P$1
- new net T8_PHS2: T8.P$2
- new net T8_PHS3: T8.P$3
- net +3V3: now also J11.5; no longer J3.5, U$2.VOUT
- net 12V: now also U$1G$2.P$A, U$1G$2.P$B, U$1G$2.P$C, U$1G$2.P$D, U$1G$2.P$E, U$1G$2.P$O, U$1G$2.P$P, U$1G$2.P$Q, U$1G$2.P$R, U$1G$2.P$S, U$2G$1.P$10, U$2G$1.P$11, U$2G$1.P$12, U$2G$1.P$13, U$2G$1.P$23, U$2G$1.P$24, U$2G$1.P$25, U$2G$1.P$26, U$2G$1.P$27, U$2G$1.P$9, U$4G$2.P$A, U$4G$2.P$B, U$4G$2.P$C, U$4G$2.P$D, U$4G$2.P$E, U$4G$2.P$O, U$4G$2.P$P, U$4G$2.P$Q, U$4G$2.P$R, U$4G$2.P$S, U$5G$1.P$10, U$5G$1.P$11, U$5G$1.P$12, U$5G$1.P$13, U$5G$1.P$23, U$5G$1.P$24, U$5G$1.P$25, U$5G$1.P$26, U$5G$1.P$27, U$5G$1.P$9, U$6G$2.P$A, U$6G$2.P$B, U$6G$2.P$C, U$6G$2.P$D, U$6G$2.P$E, U$6G$2.P$O, U$6G$2.P$P, U$6G$2.P$Q, U$6G$2.P$R, U$6G$2.P$S, U$7G$1.P$10, U$7G$1.P$11, U$7G$1.P$12, U$7G$1.P$13, U$7G$1.P$23, U$7G$1.P$24, U$7G$1.P$25, U$7G$1.P$26, U$7G$1.P$27, U$7G$1.P$9; no longer C18.+, J11.2, U$2.VIN
- net 3.3V: now also J3.5, U$1G$2.P$G, U$1G$2.P$H, U$1G$2.P$U, U$1G$2.P$V, U$4G$2.P$G, U$4G$2.P$H, U$4G$2.P$U, U$4G$2.P$V, U$6G$2.P$G, U$6G$2.P$H, U$6G$2.P$U, U$6G$2.P$V
- net CAN_H: now also U$2G$1.P$6, U$5G$1.P$6, U$7G$1.P$6; no longer J12.2
- net CAN_L: now also U$2G$1.P$7, U$5G$1.P$7, U$7G$1.P$7; no longer J12.1
- net GND: now also U$1G$2.P$AA, U$1G$2.P$BB, U$1G$2.P$J, U$1G$2.P$K, U$1G$2.P$L, U$1G$2.P$M, U$1G$2.P$N, U$1G$2.P$X, U$1G$2.P$Y, U$1G$2.P$Z, U$2G$1.P$1, U$2G$1.P$15, U$2G$1.P$16, U$2G$1.P$17, U$2G$1.P$18, U$2G$1.P$2, U$2G$1.P$3, U$2G$1.P$4, U$4G$2.P$AA, U$4G$2.P$BB, U$4G$2.P$J, U$4G$2.P$K, U$4G$2.P$L, U$4G$2.P$M, U$4G$2.P$N, U$4G$2.P$X, U$4G$2.P$Y, U$4G$2.P$Z, U$5G$1.P$1, U$5G$1.P$15, U$5G$1.P$16, U$5G$1.P$17, U$5G$1.P$18, U$5G$1.P$2, U$5G$1.P$3, U$5G$1.P$4, U$6G$2.P$AA, U$6G$2.P$BB, U$6G$2.P$J, U$6G$2.P$K, U$6G$2.P$L, U$6G$2.P$M, U$6G$2.P$N, U$6G$2.P$X, U$6G$2.P$Y, U$6G$2.P$Z, U$7G$1.P$1, U$7G$1.P$15, U$7G$1.P$16, U$7G$1.P$17, U$7G$1.P$18, U$7G$1.P$2, U$7G$1.P$3, U$7G$1.P$4; no longer C18.-, U$2.GND
- net NRST: now also J11.6, U$2G$1.P$20, U$5G$1.P$20, U$7G$1.P$20
- net PROG_1: now also J11.2, U$7G$1.P$5
- net PROG_2: now also J11.3, U$5G$1.P$5
- net PROG_3: now also J11.4, U$2G$1.P$5
- net SWCLK: no longer U$3.PA14
- net SWCLK_1: now also U$7G$1.P$22
- net SWCLK_2: now also U$5G$1.P$22
- net SWCLK_3: now also U$2G$1.P$22
- net SWCLK_IN: now also J11.7
- net SWDIO: no longer U$3.PA13
- net SWDIO_1: now also U$7G$1.P$21
- net SWDIO_2: now also U$5G$1.P$21
- net SWDIO_3: now also U$2G$1.P$21
- net SWDIO_IN: now also J11.8
Other:
- note added: "QUAD ESC CONNECTION"
- note added: "Thrusters & Motors"
- note removed: "12V to 3V3"
- note removed: "PROG_1 high and PROG_3 low chooses esc 1 PROG_1 low and PROG_3 high chooses esc 3 PROG_1 low and PROG_3 low chooses esc 2"
- note removed: "T21 Connector for 12V, CAN, GND"
- moved on the sheet: J2, J4, J5, MUX

Commit message: Design review changes-2
Parts:
- removed J10, J6, J7, J8, J9: (no value), SparkFun-Connectors:CONN_02
- added J12: 284512-8, 284512-8:284512-8
- added R5: 26.7k, SparkFun-Resistors:26.7KOHM0603-1/10W-1%
- added R8: 10k, SparkFun-Resistors:10KOHM-0603-1/10W-1%
- added R9: 5k, SparkFun-Resistors:1KOHM-0603-1/10W-1%
- J1: value (none) -> 284512-4; device SparkFun-Connectors:CONN_02 -> 284512-4:284512-4
- R10, R11: value 60 -> 1k
Connections:
- new net GPIO0: U$3.PA2
- new net N$3: R5.1
- new net N$4: R8.1
- net +3V3: no longer C1.1, C2.1, C3.1, C4.1, C5.1, C6.1, J11.5, R2.2, R6.2, SV1.5, U$3.VDD, U$3.VDDA, U$3.VDDIO2
- net 12V: now also J12.7; no longer J1.1, J10.1, J6.1, J7.1, J8.1, J9.1
- net 3.3V: now also C1.1, C2.1, C3.1, C4.1, C5.1, C6.1, J11.5, R2.2, R6.2, SV1.5, U$3.VDD, U$3.VDDA, U$3.VDDIO2
- net 5V: now also J1.1, J1.2
- net ESC-ID_1: now also R5.2
- net ESC-ID_2: now also R8.2
- net ESC-ID_3: now also R9.2
- net GND: now also J1.3, J1.4, R9.1
- net SOL1_1: now also J12.1; no longer J1.2
- net SOL2_1: now also J12.2; no longer J6.2
- net SOL3_1: now also J12.3; no longer J7.2
- net SOL4_1: now also J12.4; no longer J8.2
- net SOL5_1: now also J12.5; no longer J9.2
- net SOL6_1: now also J12.6; no longer J10.2
- net SWDIO_IN: now also J12.8
Other:
- note added: "Camera"

Commit message: added LED resistor values
Parts:
- R4, R6: value (none) -> 470
- R5: value 26.7k -> 22k
- R9: value 5k -> 4.7k
Connections:
- removed net N$4: R8.1
- net GND: now also R8.1
Changed lines of the file:
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@@
 <part name="D2" library="SparkFun-LED" library_urn="urn:adsk.eagle:library:529" deviceset="LED" device="0603" package3d_urn="urn:adsk.eagle:package:39354/1"/>
 <part name="D4" library="SparkFun-LED" library_urn="urn:adsk.eagle:library:529" deviceset="LED" device="0603" package3d_urn="urn:adsk.eagle:package:39354/1"/>
-<part name="R4" library="SparkFun-Resistors" library_urn="urn:adsk.eagle:library:532" deviceset="RESISTOR" device="0603" package3d_urn="urn:adsk.eagle:package:39650/1" value=" "/>
-<part name="R6" library="SparkFun-Resistors" library_urn="urn:adsk.eagle:library:532" deviceset="RESISTOR" device="0603" package3d_urn="urn:adsk.eagle:package:39650/1" value=" "/>
+<part name="R4" library="SparkFun-Resistors" library_urn="urn:adsk.eagle:library:532" deviceset="RESISTOR" device="0603" package3d_urn="urn:adsk.eagle:package:39650/1" value="470"/>
+<part name="R6" library="SparkFun-Resistors" library_urn="urn:adsk.eagle:library:532" deviceset="RESISTOR" device="0603" package3d_urn="urn:adsk.eagle:package:39650/1" value="470"/>
 <part name="FRAME3" library="frames" library_urn="urn:adsk.eagle:library:229" deviceset="A4L-LOC" device=""/>
 <part name="FRAME4" library="frames" library_urn="urn:adsk.eagle:library:229" deviceset="A4L-LOC" device=""/>
@@
 <part name="J12" library="284512-8" deviceset="284512-8" device=""/>
 <part name="J1" library="284512-4" deviceset="284512-4" device=""/>
-<part name="R5" library="SparkFun-Resistors" library_urn="urn:adsk.eagle:library:532" deviceset="26.7KOHM" device="0603-1/10W-1%" package3d_urn="urn:adsk.eagle:package:39650/1" value="26.7k"/>
+<part name="R5" library="SparkFun-Resistors" library_urn="urn:adsk.eagle:library:532" deviceset="26.7KOHM" device="0603-1/10W-1%" package3d_urn="urn:adsk.eagle:package:39650/1" value="22k"/>
 <part name="R8" library="SparkFun-Resistors" library_urn="urn:adsk.eagle:library:532" deviceset="10KOHM" device="-0603-1/10W-1%" package3d_urn="urn:adsk.eagle:package:39650/1" value="10k"/>
-<part name="R9" library="SparkFun-Resistors" library_urn="urn:adsk.eagle:library:532" deviceset="1KOHM" device="-0603-1/10W-1%" package3d_urn="urn:adsk.eagle:package:39650/1" value="5k"/>
+<part name="R9" library="SparkFun-Resistors" library_urn="urn:adsk.eagle:library:532" deviceset="1KOHM" device="-0603-1/10W-1%" package3d_urn="urn:adsk.eagle:package:39650/1" value="4.7k"/>
 </parts>
 <sheets>
@@
 <label x="113.03" y="115.57" size="1.778" layer="95"/>
 </segment>
+<segment>
+<pinref part="R8" gate="G$1" pin="1"/>
+<wire x1="30.48" y1="41.91" x2="30.48" y2="38.1" width="0.1524" layer="91"/>
+<label x="29.21" y="35.56" size="1.778" layer="95"/>
+</segment>
 </net>
 <net name="SWDIO_3" class="0">
@@
 </segment>
 </net>
-<net name="N$4" class="0">
-<segment>
-<pinref part="R8" gate="G$1" pin="1"/>
-<wire x1="30.48" y1="41.91" x2="30.48" y2="38.1" width="0.1524" layer="91"/>
-</segment>
-</net>

Commit message: draft board layout-  missing power connector
Parts:
- removed C1, C10, C2, C7, C8, C9: 4.7uF, SparkFun-Capacitors:4.7UF0603
- removed C11: 0.1uF, SparkFun-Capacitors:0.1UF-0603-25V-(+80/-20%)
- removed C3, C4: 100nF, SparkFun-Capacitors:4.7UF0603
- removed C5: 0.01uF, SparkFun-Capacitors:4.7UF0603
- removed C6: 1uF, SparkFun-Capacitors:4.7UF0603
- removed D1, D2, D4: (no value), SparkFun-LED:LED0603
- removed J11, J12: 284512-8, 284512-8:284512-8
- removed R10, R11: 1k, SparkFun-Resistors:1KOHM-0603-1/10W-1%
- removed R4, R6: 470, SparkFun-Resistors:RESISTOR0603
- removed R5: 22k, SparkFun-Resistors:26.7KOHM0603-1/10W-1%
- removed R7: (no value), SparkFun-Resistors:RESISTOR0603
- removed R8: 10k, SparkFun-Resistors:10KOHM-0603-1/10W-1%
- removed R9: 4.7k, SparkFun-Resistors:1KOHM-0603-1/10W-1%
- removed RESET: SWITCH, DiscreteComponents:SWITCH
- removed SV1: (no value), con-lsta:FE05-1
- removed U$1, U$2, U$4, U$5, U$6: ESC2BACKPLANE, ESC_to_Backplane_Connectors:ESC2BACKPLANE
- removed U1: ULN2003V12, ULN2003V12:ULN2003V12
- removed Y1: ECS-80-S-4X, ECS-80-S-4X:ECS-80-S-4X
- R1: value 1k -> 22k; device SparkFun-Resistors:1KOHM-0603-1/10W-1% -> SparkFun-Resistors:26.7KOHM0603-1/10W-1%
- R2: value 1k -> 10k; device SparkFun-Resistors:1KOHM-0603-1/10W-1% -> SparkFun-Resistors:10KOHM-0603-1/10W-1%
- R3: value 1k -> 4.7k
- U$3: value STM32F042K6T6 -> ESC2BACKPLANE; device PI_Shield_Library:STM32F042K6T6 -> ESC_to_Backplane_Connectors:ESC2BACKPLANE
- U$8: value TCAN337D -> ESC2BACKPLANE; device PI_Shield_Library:TCAN337D -> ESC_to_Backplane_Connectors:ESC2BACKPLANE
Connections:
- removed net +3V3: C10.1, U$8.VCC
- removed net ALERT: U$3.PB7
- removed net CAN_RX: U$3.PA11, U$8.RXD
- removed net CAN_TX: U$3.PA12, U$8.TXD
- removed net CLK: U$3.PA9
- removed net DATA: U$3.PA10
- removed net GPIO0: U$3.PA2
- removed net GPIO1: U$3.PB6, U1.IN4
- removed net GPIO10: U$3.PA5, U1.IN3
- removed net GPIO11: U$3.PA6, U1.IN2
- removed net GPIO12: U$3.PA7, U1.IN1
- removed net GPIO13: U$3.PA8
- removed net GPIO14: U$3.PA1
- removed net GPIO15: U$3.PA0
- removed net GPIO2: U$3.PB4, U1.IN5
- removed net GPIO3: U$3.PB3, U1.IN6
- removed net GPIO8: U$3.PA3
- removed net GPIO9: U$3.PA4
- removed net LED: R7.2, U$3.PA15
- removed net N$1: C9.1, R1.1, Y1.2
- removed net N$2: C8.1, R3.1, Y1.1
- removed net N$24: D1.A, R7.1
- removed net N$25: D4.A, R4.1
- removed net N$27: D2.A, R6.1
- removed net N$3: R5.1
- removed net N$5: C11.2, R10.1, R11.2
- removed net OSC_IN: R3.2, U$3.PF0-OSC_IN
- removed net OSC_OUT: R1.2, U$3.PF1-OSC_OUT
- removed net SOL1_1: J12.1, U1.OUT1
- removed net SOL2_1: J12.2, U1.OUT2
- removed net SOL3_1: J12.3, U1.OUT3
- removed net SOL4_1: J12.4, U1.OUT4
- removed net SOL5_1: J12.5, U1.OUT5
- removed net SOL6_1: J12.6, U1.OUT6
- removed net SWCLK: SV1.4
- removed net SWDIO: SV1.2
- net 12V: now also U$3G$1.P$10, U$3G$1.P$11, U$3G$1.P$12, U$3G$1.P$13, U$3G$1.P$9, U$3G$2.P$A, U$3G$2.P$B, U$3G$2.P$C, U$3G$2.P$D, U$3G$2.P$E, U$3G$2.P$O, U$3G$2.P$P, U$3G$2.P$Q, U$3G$2.P$R, U$3G$2.P$S, U$7G$2.P$A, U$7G$2.P$B, U$7G$2.P$C, U$7G$2.P$D, U$7G$2.P$E, U$7G$2.P$O, U$7G$2.P$P, U$7G$2.P$Q, U$7G$2.P$R, U$7G$2.P$S, U$8G$1.P$10, U$8G$1.P$11, U$8G$1.P$12, U$8G$1.P$13, U$8G$1.P$9, U$8G$2.P$A, U$8G$2.P$B, U$8G$2.P$C, U$8G$2.P$D, U$8G$2.P$E, U$8G$2.P$O, U$8G$2.P$P, U$8G$2.P$Q, U$8G$2.P$R, U$8G$2.P$S; no longer J12.7, R4.2, U$1G$2.P$A, U$1G$2.P$B, U$1G$2.P$C, U$1G$2.P$D, U$1G$2.P$E, U$1G$2.P$O, U$1G$2.P$P, U$1G$2.P$Q, U$1G$2.P$R, U$1G$2.P$S, U$2G$1.P$10, U$2G$1.P$11, U$2G$1.P$12, U$2G$1.P$13, U$2G$1.P$23, U$2G$1.P$24, U$2G$1.P$25, U$2G$1.P$26, U$2G$1.P$27, U$2G$1.P$9, U$4G$2.P$A, U$4G$2.P$B, U$4G$2.P$C, U$4G$2.P$D, U$4G$2.P$E, U$4G$2.P$O, U$4G$2.P$P, U$4G$2.P$Q, U$4G$2.P$R, U$4G$2.P$S, U$5G$1.P$10, U$5G$1.P$11, U$5G$1.P$12, U$5G$1.P$13, U$5G$1.P$23, U$5G$1.P$24, U$5G$1.P$25, U$5G$1.P$26, U$5G$1.P$27, U$5G$1.P$9, U$6G$2.P$A, U$6G$2.P$B, U$6G$2.P$C, U$6G$2.P$D, U$6G$2.P$E, U$6G$2.P$O, U$6G$2.P$P, U$6G$2.P$Q, U$6G$2.P$R, U$6G$2.P$S, U$7G$1.P$23, U$7G$1.P$24, U$7G$1.P$25, U$7G$1.P$26, U$7G$1.P$27, U1.COM
- net 3.3V: now also U$3G$2.P$G, U$3G$2.P$H, U$3G$2.P$U, U$3G$2.P$V, U$7G$2.P$G, U$7G$2.P$H, U$7G$2.P$U, U$7G$2.P$V, U$8G$2.P$G, U$8G$2.P$H, U$8G$2.P$U, U$8G$2.P$V; no longer C1.1, C2.1, C3.1, C4.1, C5.1, C6.1, J11.5, R2.2, R6.2, SV1.5, U$1G$2.P$G, U$1G$2.P$H, U$1G$2.P$U, U$1G$2.P$V, U$3.VDD, U$3.VDDA, U$3.VDDIO2, U$4G$2.P$G, U$4G$2.P$H, U$4G$2.P$U, U$4G$2.P$V, U$6G$2.P$G, U$6G$2.P$H, U$6G$2.P$U, U$6G$2.P$V
- net CAN_H: now also U$3G$1.P$6, U$8G$1.P$6; no longer R10.2, U$2G$1.P$6, U$5G$1.P$6, U$8.CANH
- net CAN_L: now also U$3G$1.P$7, U$8G$1.P$7; no longer R11.1, U$2G$1.P$7, U$5G$1.P$7, U$8.CANL
- net ESC-ID_1: now also R1.2, U$3G$1.P$8; no longer R5.2, U$7G$1.P$8
- net ESC-ID_2: now also R2.2, U$7G$1.P$8; no longer R8.2, U$5G$1.P$8
- net ESC-ID_3: now also R3.2, U$8G$1.P$8; no longer R9.2, U$2G$1.P$8
- net GND: now also R1.1, R2.1, R3.1, U$3G$1.P$1, U$3G$1.P$15, U$3G$1.P$16, U$3G$1.P$17, U$3G$1.P$18, U$3G$1.P$2, U$3G$1.P$23, U$3G$1.P$24, U$3G$1.P$25, U$3G$1.P$26, U$3G$1.P$27, U$3G$1.P$3, U$3G$1.P$4, U$3G$2.P$AA, U$3G$2.P$BB, U$3G$2.P$J, U$3G$2.P$K, U$3G$2.P$L, U$3G$2.P$M, U$3G$2.P$N, U$3G$2.P$X, U$3G$2.P$Y, U$3G$2.P$Z, U$7G$1.P$23, U$7G$1.P$24, U$7G$1.P$25, U$7G$1.P$26, U$7G$1.P$27, U$7G$2.P$AA, U$7G$2.P$BB, U$7G$2.P$J, U$7G$2.P$K, U$7G$2.P$L, U$7G$2.P$M, U$7G$2.P$N, U$7G$2.P$X, U$7G$2.P$Y, U$7G$2.P$Z, U$8G$1.P$1, U$8G$1.P$15, U$8G$1.P$16, U$8G$1.P$17, U$8G$1.P$18, U$8G$1.P$2, U$8G$1.P$23, U$8G$1.P$24, U$8G$1.P$25, U$8G$1.P$26, U$8G$1.P$27, U$8G$1.P$3, U$8G$1.P$4, U$8G$2.P$AA, U$8G$2.P$BB, U$8G$2.P$J, U$8G$2.P$K, U$8G$2.P$L, U$8G$2.P$M, U$8G$2.P$N, U$8G$2.P$X, U$8G$2.P$Y, U$8G$2.P$Z; no longer C1.2, C10.2, C11.1, C2.2, C3.2, C4.2, C5.2, C6.2, C7.2, C8.2, C9.2, D1.C, D2.C, D4.C, J11.1, R8.1, R9.1, RESET.P$1, SV1.3, U$1G$2.P$AA, U$1G$2.P$BB, U$1G$2.P$J, U$1G$2.P$K, U$1G$2.P$L, U$1G$2.P$M, U$1G$2.P$N, U$1G$2.P$X, U$1G$2.P$Y, U$1G$2.P$Z, U$2G$1.P$1, U$2G$1.P$15, U$2G$1.P$16, U$2G$1.P$17, U$2G$1.P$18, U$2G$1.P$2, U$2G$1.P$3, U$2G$1.P$4, U$3.PB8-BOOT0, U$3.VSS, U$3.VSS1, U$4G$2.P$AA, U$4G$2.P$BB, U$4G$2.P$J, U$4G$2.P$K, U$4G$2.P$L, U$4G$2.P$M, U$4G$2.P$N, U$4G$2.P$X, U$4G$2.P$Y, U$4G$2.P$Z, U$5G$1.P$1, U$5G$1.P$15, U$5G$1.P$16, U$5G$1.P$17, U$5G$1.P$18, U$5G$1.P$2, U$5G$1.P$3, U$5G$1.P$4, U$6G$2.P$AA, U$6G$2.P$BB, U$6G$2.P$J, U$6G$2.P$K, U$6G$2.P$L, U$6G$2.P$M, U$6G$2.P$N, U$6G$2.P$X, U$6G$2.P$Y, U$6G$2.P$Z, U$8.GND, U1.GND
- net NRST: now also U$3G$1.P$20, U$8G$1.P$20; no longer C7.1, J11.6, R2.1, RESET.P$2, SV1.1, U$2G$1.P$20, U$3.NRST, U$5G$1.P$20
- net PROG_1: now also U$3G$1.P$5; no longer J11.2, U$7G$1.P$5
- net PROG_2: now also U$7G$1.P$5; no longer J11.3, U$5G$1.P$5
- net PROG_3: now also U$8G$1.P$5; no longer J11.4, U$2G$1.P$5
- net SWCLK_1: now also U$3G$1.P$22; no longer U$7G$1.P$22
- net SWCLK_2: now also U$7G$1.P$22; no longer U$5G$1.P$22
- net SWCLK_3: now also U$8G$1.P$22; no longer U$2G$1.P$22
- net SWCLK_4: no longer U$3.PA14
- net SWCLK_IN: no longer J11.7
- net SWDIO_1: now also U$3G$1.P$21; no longer U$7G$1.P$21
- net SWDIO_2: now also U$7G$1.P$21; no longer U$5G$1.P$21
- net SWDIO_3: now also U$8G$1.P$21; no longer U$2G$1.P$21
- net SWDIO_4: no longer U$3.PA13
- net SWDIO_IN: no longer J11.8, J12.8
Other:
- note removed: "CAN"
- note removed: "CAN TERMINATION"
- note removed: "CAN TRANSCEIVER"
- note removed: "NPN Array"
- note removed: "OUTPUT HEADERS"
- note removed: "Pin 1 (VDD)"
- note removed: "Pin 17 (VDDIO2)"
- note removed: "Pin 5 (VDDA)"
- note removed: "Power Indication LEDs"
- note removed: "STM"

Commit message: added back solenoid board
Parts:
- added C1, C10, C2, C7, C8, C9: 4.7uF, SparkFun-Capacitors:4.7UF0603
- added C11: 0.1uF, SparkFun-Capacitors:0.1UF-0603-25V-(+80/-20%)
- added C3, C4: 100nF, SparkFun-Capacitors:4.7UF0603
- added C5: 0.01uF, SparkFun-Capacitors:4.7UF0603
- added C6: 1uF, SparkFun-Capacitors:4.7UF0603
- added D1, D2, D4: (no value), SparkFun-LED:LED0603
- added J11, J12: 284512-8, 284512-8:284512-8
- added R10, R11, R5, R7, R8: 1k, SparkFun-Resistors:1KOHM-0603-1/10W-1%
- added R4, R6: 470, SparkFun-Resistors:RESISTOR0603
- added R9: (no value), SparkFun-Resistors:RESISTOR0603
- added RESET: SWITCH, DiscreteComponents:SWITCH
- added SV1: (no value), con-lsta:FE05-1
- added U$1: TCAN337D, PI_Shield_Library:TCAN337D
- added U$2: STM32F042K6T6, PI_Shield_Library:STM32F042K6T6
- added U1: ULN2003V12, ULN2003V12:ULN2003V12
- added Y1: ECS-80-S-4X, ECS-80-S-4X:ECS-80-S-4X
Connections:
- new net +3V3: C10.1, U$1.VCC
- new net ALERT1: U$2.PB7
- new net ALERT2: U$2.PB5
- new net C2_1: U$2.PB0
- new net C2_2: U$2.PB1
- new net CAN_RX: U$1.RXD, U$2.PA11
- new net CAN_TX: U$1.TXD, U$2.PA12
- new net CLK: U$2.PA9
- new net DATA: U$2.PA10
- new net GPIO0: U$2.PA2
- new net GPIO1: U$2.PB6, U1.IN4
- new net GPIO10: U$2.PA5, U1.IN3
- new net GPIO11: U$2.PA6, U1.IN2
- new net GPIO12: U$2.PA7, U1.IN1
- new net GPIO13: U$2.PA8
- new net GPIO14: U$2.PA1
- new net GPIO15: U$2.PA0
- new net GPIO2: U$2.PB4, U1.IN5
- new net GPIO3: U$2.PB3, U1.IN6
- new net GPIO8: U$2.PA3
- new net GPIO9: U$2.PA4
- new net LED: R9.2, U$2.PA15
- new net N$1: C9.1, R5.1, Y1.2
- new net N$2: C8.1, R8.1, Y1.1
- new net N$24: D1.A, R9.1
- new net N$25: D4.A, R4.1
- new net N$27: D2.A, R6.1
- new net N$5: C11.2, R10.1, R11.2
- new net OSC_IN: R8.2, U$2.PF0-OSC_IN
- new net OSC_OUT: R5.2, U$2.PF1-OSC_OUT
- new net PROG_4: J11.2
- new net SOL1_1: J12.1, U1.OUT1
- new net SOL2_1: J12.2, U1.OUT2
- new net SOL3_1: J12.3, U1.OUT3
- new net SOL4_1: J12.4, U1.OUT4
- new net SOL5_1: J12.5, U1.OUT5
- new net SOL6_1: J12.6, U1.OUT6
- new net SWCLK: SV1.4
- new net SWDIO: SV1.2
- net 12V: now also J12.7, R4.2, U$3G$1.P$23, U$3G$1.P$24, U$3G$1.P$25, U$3G$1.P$26, U$3G$1.P$27, U$7G$1.P$23, U$7G$1.P$24, U$7G$1.P$25, U$7G$1.P$26, U$7G$1.P$27, U$8G$1.P$23, U$8G$1.P$24, U$8G$1.P$25, U$8G$1.P$26, U$8G$1.P$27, U1.COM
- net 3.3V: now also C1.1, C2.1, C3.1, C4.1, C5.1, C6.1, J11.5, R6.2, R7.2, SV1.5, U$2.VDD, U$2.VDDA, U$2.VDDIO2
- net CAN_H: now also R10.2, U$1.CANH
- net CAN_L: now also R11.1, U$1.CANL
- net GND: now also C1.2, C10.2, C11.1, C2.2, C3.2, C4.2, C5.2, C6.2, C7.2, C8.2, C9.2, D1.C, D2.C, D4.C, J11.1, RESET.P$1, SV1.3, U$1.GND, U$2.PB8-BOOT0, U$2.VSS, U$2.VSS1, U1.GND; no longer U$3G$1.P$23, U$3G$1.P$24, U$3G$1.P$25, U$3G$1.P$26, U$3G$1.P$27, U$7G$1.P$23, U$7G$1.P$24, U$7G$1.P$25, U$7G$1.P$26, U$7G$1.P$27, U$8G$1.P$23, U$8G$1.P$24, U$8G$1.P$25, U$8G$1.P$26, U$8G$1.P$27
- net NRST: now also C7.1, J11.6, R7.1, RESET.P$2, SV1.1, U$2.NRST
- net PROG_2: now also J11.3
- net PROG_3: now also J11.4
- net SWCLK_4: now also U$2.PA14
- net SWCLK_IN: now also J11.7
- net SWDIO_4: now also U$2.PA13
- net SWDIO_IN: now also J11.8, J12.8
Other:
- note added: "CAN"
- note added: "CAN TERMINATION"
- note added: "CAN TRANSCEIVER"
- note added: "NPN Array"
- note added: "OUTPUT HEADERS"
- note added: "Pin 1 (VDD)"
- note added: "Pin 17 (VDDIO2)"
- note added: "Pin 5 (VDDA)"
- note added: "Power Indication LEDs"
- note added: "STM"

Commit message: removed solenoid board
Parts:
- removed C1, C10, C2, C7, C8, C9: 4.7uF, SparkFun-Capacitors:4.7UF0603
- removed C11: 0.1uF, SparkFun-Capacitors:0.1UF-0603-25V-(+80/-20%)
- removed C3, C4: 100nF, SparkFun-Capacitors:4.7UF0603
- removed C5: 0.01uF, SparkFun-Capacitors:4.7UF0603
- removed C6: 1uF, SparkFun-Capacitors:4.7UF0603
- removed D1, D2, D4: (no value), SparkFun-LED:LED0603
- removed J11, J12: 284512-8, 284512-8:284512-8
- removed R10, R11, R5, R7, R8: 1k, SparkFun-Resistors:1KOHM-0603-1/10W-1%
- removed R4, R6: 470, SparkFun-Resistors:RESISTOR0603
- removed R9: (no value), SparkFun-Resistors:RESISTOR0603
- removed RESET: SWITCH, DiscreteComponents:SWITCH
- removed SV1: (no value), con-lsta:FE05-1
- removed U$1: TCAN337D, PI_Shield_Library:TCAN337D
- removed U$2: STM32F042K6T6, PI_Shield_Library:STM32F042K6T6
- removed U1: ULN2003V12, ULN2003V12:ULN2003V12
- removed Y1: ECS-80-S-4X, ECS-80-S-4X:ECS-80-S-4X
Connections:
- removed net +3V3: C10.1, U$1.VCC
- removed net ALERT1: U$2.PB7
- removed net ALERT2: U$2.PB5
- removed net C2_1: U$2.PB0
- removed net C2_2: U$2.PB1
- removed net CAN_RX: U$1.RXD, U$2.PA11
- removed net CAN_TX: U$1.TXD, U$2.PA12
- removed net CLK: U$2.PA9
- removed net DATA: U$2.PA10
- removed net GPIO0: U$2.PA2
- removed net GPIO1: U$2.PB6, U1.IN4
- removed net GPIO10: U$2.PA5, U1.IN3
- removed net GPIO11: U$2.PA6, U1.IN2
- removed net GPIO12: U$2.PA7, U1.IN1
- removed net GPIO13: U$2.PA8
- removed net GPIO14: U$2.PA1
- removed net GPIO15: U$2.PA0
- removed net GPIO2: U$2.PB4, U1.IN5
- removed net GPIO3: U$2.PB3, U1.IN6
- removed net GPIO8: U$2.PA3
- removed net GPIO9: U$2.PA4
- removed net LED: R9.2, U$2.PA15
- removed net N$1: C9.1, R5.1, Y1.2
- removed net N$2: C8.1, R8.1, Y1.1
- removed net N$24: D1.A, R9.1
- removed net N$25: D4.A, R4.1
- removed net N$27: D2.A, R6.1
- removed net N$5: C11.2, R10.1, R11.2
- removed net OSC_IN: R8.2, U$2.PF0-OSC_IN
- removed net OSC_OUT: R5.2, U$2.PF1-OSC_OUT
- removed net PROG_4: J11.2
- removed net SOL1_1: J12.1, U1.OUT1
- removed net SOL2_1: J12.2, U1.OUT2
- removed net SOL3_1: J12.3, U1.OUT3
- removed net SOL4_1: J12.4, U1.OUT4
- removed net SOL5_1: J12.5, U1.OUT5
- removed net SOL6_1: J12.6, U1.OUT6
- removed net SWCLK: SV1.4
- removed net SWDIO: SV1.2
- net 12V: no longer J12.7, R4.2, U1.COM
- net 3.3V: no longer C1.1, C2.1, C3.1, C4.1, C5.1, C6.1, J11.5, R6.2, R7.2, SV1.5, U$2.VDD, U$2.VDDA, U$2.VDDIO2
- net CAN_H: no longer R10.2, U$1.CANH
- net CAN_L: no longer R11.1, U$1.CANL
- net GND: no longer C1.2, C10.2, C11.1, C2.2, C3.2, C4.2, C5.2, C6.2, C7.2, C8.2, C9.2, D1.C, D2.C, D4.C, J11.1, RESET.P$1, SV1.3, U$1.GND, U$2.PB8-BOOT0, U$2.VSS, U$2.VSS1, U1.GND
- net NRST: no longer C7.1, J11.6, R7.1, RESET.P$2, SV1.1, U$2.NRST
- net PROG_2: no longer J11.3
- net PROG_3: no longer J11.4
- net SWCLK_4: no longer U$2.PA14
- net SWCLK_IN: no longer J11.7
- net SWDIO_4: no longer U$2.PA13
- net SWDIO_IN: no longer J11.8, J12.8
Other:
- note removed: "CAN"
- note removed: "CAN TERMINATION"
- note removed: "CAN TRANSCEIVER"
- note removed: "NPN Array"
- note removed: "OUTPUT HEADERS"
- note removed: "Pin 1 (VDD)"
- note removed: "Pin 17 (VDDIO2)"
- note removed: "Pin 5 (VDDA)"
- note removed: "Power Indication LEDs"
- note removed: "STM"
